File: PCBs/power-supply.brd (EAGLE design)
At the start: 210.5 x 118.1 mm, 46 parts, among them U3 TL783

Commit message: Started amp.
Parts:
- added PAD17: +310V-R, wirepad:3,81/1,4
- added PAD18: +310V-L, wirepad:3,81/1,4
- added PAD19, PAD21: 0V, wirepad:3,81/1,4
- added PAD20: +38V, wirepad:3,81/1,4
- added PAD22: -38V, wirepad:3,81/1,4
Connections:
- net GND: now also PAD19.1
- net GND2: now also PAD21.1
- net N$10: now also PAD20.1
- net N$13: now also PAD22.1
- net N$3: now also PAD17.1
- net N$7: now also PAD18.1
Changed lines of the file:
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@@
 <element name="U$1" library="mugen" package="WOG" value="W10G" x="-45.72" y="111.76"/>
 <element name="U3" library="linear" library_urn="urn:adsk.eagle:library:262" package="TO220V" package3d_urn="urn:adsk.eagle:package:16417/1" value="TL783" x="-71.12" y="114.3"/>
+<element name="PAD17" library="wirepad" library_urn="urn:adsk.eagle:library:412" package="3,81/1,4" package3d_urn="urn:adsk.eagle:package:30835/1" value="+310V-R" x="-114.3" y="-30.48"/>
+<element name="PAD18" library="wirepad" library_urn="urn:adsk.eagle:library:412" package="3,81/1,4" package3d_urn="urn:adsk.eagle:package:30835/1" value="+310V-L" x="-114.3" y="-68.58"/>
+<element name="PAD19" library="wirepad" library_urn="urn:adsk.eagle:library:412" package="3,81/1,4" package3d_urn="urn:adsk.eagle:package:30835/1" value="0V" x="-114.3" y="-106.68"/>
+<element name="PAD20" library="wirepad" library_urn="urn:adsk.eagle:library:412" package="3,81/1,4" package3d_urn="urn:adsk.eagle:package:30835/1" value="+38V" x="106.68" y="68.58"/>
+<element name="PAD21" library="wirepad" library_urn="urn:adsk.eagle:library:412" package="3,81/1,4" package3d_urn="urn:adsk.eagle:package:30835/1" value="0V" x="114.3" y="33.02"/>
+<element name="PAD22" library="wirepad" library_urn="urn:adsk.eagle:library:412" package="3,81/1,4" package3d_urn="urn:adsk.eagle:package:30835/1" value="-38V" x="106.68" y="7.62"/>
 </elements>
 <signals>
@@
 <contactref element="C27" pad="+"/>
 <contactref element="PAD3" pad="1"/>
-<wire x1="-90.17" y1="130.81" x2="-13.97" y2="137.16" width="0" layer="19" extent="1-1"/>
-<wire x1="-72.39" y1="81.28" x2="-90.17" y2="130.81" width="0" layer="19" extent="1-1"/>
+<contactref element="PAD17" pad="1"/>
+<wire x1="-72.39" y1="81.28" x2="-114.3" y2="-30.48" width="0" layer="19" extent="1-1"/>
+<wire x1="-90.17" y1="130.81" x2="-72.39" y2="81.28" width="0" layer="19" extent="1-1"/>
+<wire x1="-13.97" y1="137.16" x2="-90.17" y2="130.81" width="0" layer="19" extent="1-1"/>
 </signal>
 <signal name="N$7">
@@
 <contactref element="C28" pad="+"/>
 <contactref element="PAD4" pad="1"/>
-<wire x1="-96.52" y1="130.81" x2="-29.21" y2="137.16" width="0" layer="19" extent="1-1"/>
-<wire x1="-91.44" y1="81.28" x2="-96.52" y2="130.81" width="0" layer="19" extent="1-1"/>
+<contactref element="PAD18" pad="1"/>
+<wire x1="-91.44" y1="81.28" x2="-114.3" y2="-68.58" width="0" layer="19" extent="1-1"/>
+<wire x1="-96.52" y1="130.81" x2="-91.44" y2="81.28" width="0" layer="19" extent="1-1"/>
+<wire x1="-29.21" y1="137.16" x2="-96.52" y2="130.81" width="0" layer="19" extent="1-1"/>
 </signal>
 <signal name="N$8">
@@
 <wire x1="12.7" y1="66.04" x2="10.16" y2="63.5" width="1.27" layer="1"/>
 <wire x1="12.7" y1="69.723" x2="12.7" y2="63.5" width="1.27" layer="1"/>
+<contactref element="PAD20" pad="1"/>
+<wire x1="106.68" y1="68.58" x2="112.08" y2="68.81" width="0" layer="19" extent="1-1"/>
 <wire x1="114.3" y1="63.5" x2="112.08" y2="68.81" width="0" layer="19" extent="1-1"/>
 </signal>
@@
 <wire x1="12.7" y1="12.7" x2="10.16" y2="15.24" width="1.27" layer="1"/>
 <wire x1="12.7" y1="9.017" x2="12.7" y2="15.24" width="1.27" layer="1"/>
+<contactref element="PAD22" pad="1"/>
+<wire x1="106.68" y1="7.62" x2="112.5" y2="7.81" width="0" layer="19" extent="1-1"/>
 <wire x1="114.3" y1="15.24" x2="112.5" y2="7.81" width="0" layer="19" extent="1-1"/>
 </signal>
@@
 <contactref element="C28" pad="-"/>
 <contactref element="C27" pad="-"/>
-<wire x1="-22.86" y1="83.82" x2="-17.78" y2="99.568" width="0" layer="19" extent="1-1"/>
-<wire x1="-45.72" y1="82.55" x2="-22.86" y2="83.82" width="0" layer="19" extent="1-1"/>
+<contactref element="PAD19" pad="1"/>
+<wire x1="-86.36" y1="81.28" x2="-114.3" y2="-106.68" width="0" layer="19" extent="1-1"/>
+<wire x1="-67.31" y1="81.28" x2="-86.36" y2="81.28" width="0" layer="19" extent="1-1"/>
+<wire x1="-45.72" y1="82.55" x2="-67.31" y2="81.28" width="0" layer="19" extent="1-1"/>
 <wire x1="-43.18" y1="99.568" x2="-45.72" y2="82.55" width="0" layer="19" extent="1-1"/>
-<wire x1="-67.31" y1="81.28" x2="-45.72" y2="82.55" width="0" layer="19" extent="1-1"/>
-<wire x1="-86.36" y1="81.28" x2="-67.31" y2="81.28" width="0" layer="19" extent="1-1"/>
+<wire x1="-22.86" y1="83.82" x2="-45.72" y2="82.55" width="0" layer="19" extent="1-1"/>
+<wire x1="-17.78" y1="99.568" x2="-22.86" y2="83.82" width="0" layer="19" extent="1-1"/>
 <wire x1="-53.34" y1="121.92" x2="-43.18" y2="99.568" width="0" layer="19" extent="1-1"/>
 <wire x1="-78.74" y1="121.92" x2="-53.34" y2="121.92" width="0" layer="19" extent="1-1"/>
@@
 <wire x1="12.7" y1="27.94" x2="10.16" y2="25.4" width="1.27" layer="1"/>
 <wire x1="12.7" y1="31.623" x2="12.7" y2="25.4" width="1.27" layer="1"/>
+<contactref element="PAD21" pad="1"/>
+<wire x1="114.3" y1="33.02" x2="111.73" y2="39.81" width="0" layer="19" extent="1-1"/>
+<wire x1="114.3" y1="25.4" x2="114.3" y2="33.02" width="0" layer="19" extent="1-1"/>
 <wire x1="114.3" y1="53.34" x2="111.73" y2="39.81" width="0" layer="19" extent="1-1"/>
-<wire x1="114.3" y1="25.4" x2="111.73" y2="39.81" width="0" layer="19" extent="1-1"/>
 </signal>
 </signals>

Commit message: Basic design done.
Parts:
- added PAD23: +42V, wirepad:3,81/1,4
- added PAD24: 0V, wirepad:3,81/1,4
- moved PAD5 237.5 mm to (97.8, 3.81)
- moved PAD4 236.4 mm to (102.9, 3.81)
- moved PAD3 235.3 mm to (108.0, 3.81)
- moved D11 217.3 mm to (99.1, 118.1), turned to 180 degrees
- moved D13 213.9 mm to (86.4, 63.5), turned to 270 degrees
- moved D1 204.1 mm to (90.2, 63.5), turned to 270 degrees
- moved D10 200.7 mm to (99.1, 108.0)
- moved C25 199.0 mm to (108.0, 91.4), turned to 270 degrees
- moved PAD7 190.6 mm to (74.9, 137.2)
- moved PAD6 189.3 mm to (80.0, 137.2)
- moved PAD2 185.5 mm to (101.6, 137.2)
- moved D9 184.2 mm to (99.1, 113.0), turned to 180 degrees
- moved C27 183.3 mm to (101.6, 16.5), turned to 180 degrees
- moved PAD15 182.3 mm to (74.9, 3.81)
- moved C28 182.1 mm to (81.3, 16.5)
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Connections:
- net GND1: now also PAD24.1
- net N$15: now also PAD23.1
Routing:
- net GND: track 0.00 -> 127.4 mm
- net N$15: track 0.00 -> 100.7 mm
- net GND1: track 0.00 -> 95.7 mm
- net N$6: track 0.00 -> 58.6 mm
- net N$1: track 0.00 -> 46.8 mm
- net N$2: track 0.00 -> 46.6 mm
- net N$4: track 0.00 -> 38.7 mm
- net GND2: track 252.7 -> 284.4 mm
- net N$5: track 0.00 -> 21.2 mm
- net N$9: track 0.00 -> 18.6 mm
- net N$3: track 0.00 -> 18.4 mm
- net N$8: track 0.00 -> 11.5 mm
- net N$7: track 0.00 -> 11.0 mm
- net N$10: track 128.1 -> 128.9 mm
Other:
- board size 210.5 x 118.1 mm -> 111.8 x 141 mm
